File: 9key/9key_rev0.1a.brd (EAGLE design)
At the start: 160 x 100 mm, 11 parts, among them U1 PIC32MK1024MCF100100TQFP

Commit message: added keys!!!
Parts:
- added C10, C9: 22pF, resistor:C0603
- added ICSP: (no value), con-lsta:FE06
- added Q1: (no value), crystal-geyer_V1_0:3.2X2.5_KX-7
- moved C8 34.1 mm to (4.00, 5.00)
- moved C7 30.1 mm to (4.00, 7.00)
- moved C6 29.3 mm to (19.0, 7.87)
- moved R2 26.3 mm to (17.9, 11.0), turned to 90 degrees
- moved R1 23.4 mm to (20.0, 11.0), turned to 90 degrees
- moved C4 2.24 mm to (42.0, 25.0), turned to 270 degrees
- moved C3 0.07 mm to (33.0, 37.9), turned to 90 degrees
Connections:
- new net NC1: ICSP.6
- new net OSCIN: C10.1, Q1.1, U1.63
- new net OSCOUT: C9.1, Q1.3, U1.64
- new net PGEC1: ICSP.2, U1.26
- new net PGED1: ICSP.3, U1.27
- net +3V3: now also ICSP.4
- net GND: now also C10.2, C9.2, ICSP.5
- net MCLR: now also ICSP.1
Routing:
- net MCLR: track 0.00 -> 19.9 mm, vias 0 -> 2
- net +3V3: track 0.00 -> 13.0 mm
- net PGEC1: track 0.00 -> 12.8 mm
- net PGED1: track 0.00 -> 12.1 mm
- net OSCOUT: track 0.00 -> 7.62 mm
- net OSCIN: track 0.00 -> 7.17 mm
- net N$5: track 0.00 -> 4.38 mm
