File: 9key/9key_rev0.1a.sch (EAGLE design)
At the start: 11 parts, among them U1 PIC32MK1024MCF100100TQFP

Commit message: added keys!!!
Parts:
- added C10, C9: 22pF, resistor:C-USC0603
- added ICSP: (no value), con-lsta:FE06-1
- added Q1: (no value), crystal-geyer_V1_0:KX-7
Connections:
- new net NC1: ICSP.6
- new net OSCIN: C10.1, Q1.1, U1.OSCI/CLKI/AN49/CVD49/RPC12/RC12
- new net OSCOUT: C9.1, Q1.2, U1.OSCO/CLKO/RPC15/RC15
- new net PGEC1: ICSP.2, U1.PGEC1/OA1IN+/AN4/C1IN1+/C1IN3-/C2IN3-/RPB2/RB2
- new net PGED1: ICSP.3, U1.PGED1/OA1IN-/AN5/CTCMP/C1IN1-/RTCC/RPB3/RB3
- net +3V3: now also ICSP.4
- net GND: now also C10.2, C9.2, ICSP.5
- net MCLR: now also ICSP.1
Changed lines of the file:
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@@
 <part name="+3V5" library="supply1" library_urn="urn:adsk.eagle:library:371" deviceset="+3V3" device=""/>
 <part name="GND5" library="supply1" library_urn="urn:adsk.eagle:library:371" deviceset="GND" device=""/>
+<part name="ICSP" library="con-lsta" library_urn="urn:adsk.eagle:library:161" deviceset="FE06-1" device="" package3d_urn="urn:adsk.eagle:package:8191/1"/>
+<part name="Q1" library="crystal-geyer_V1_0" library_urn="urn:adsk.eagle:library:203" deviceset="KX" device="-7" package3d_urn="urn:adsk.eagle:package:11924/1"/>
+<part name="C9" library="resistor" library_urn="urn:adsk.eagle:library:348" deviceset="C-US" device="C0603" package3d_urn="urn:adsk.eagle:package:26138/1" value="22pF"/>
+<part name="C10" library="resistor" library_urn="urn:adsk.eagle:library:348" deviceset="C-US" device="C0603" package3d_urn="urn:adsk.eagle:package:26138/1" value="22pF"/>
+<part name="GND6" library="supply1" library_urn="urn:adsk.eagle:library:371" deviceset="GND" device=""/>
 </parts>
 <sheets>
@@
 <instance part="+3V5" gate="G$1" x="129.54" y="266.7"/>
 <instance part="GND5" gate="1" x="129.54" y="243.84"/>
+<instance part="ICSP" gate="G$1" x="20.32" y="157.48" rot="MR180"/>
+<instance part="Q1" gate="G$1" x="279.4" y="175.26" rot="MR270"/>
+<instance part="C9" gate="G$1" x="284.48" y="170.18" rot="R90"/>
+<instance part="C10" gate="G$1" x="284.48" y="180.34" rot="R90"/>
+<instance part="GND6" gate="1" x="292.1" y="165.1"/>
 </instances>
 <busses>
@@
 <junction x="129.54" y="248.92"/>
 <pinref part="GND5" gate="1" pin="GND"/>
+</segment>
+<segment>
+<pinref part="ICSP" gate="G$1" pin="5"/>
+<wire x1="27.94" y1="152.4" x2="40.64" y2="152.4" width="0.1524" layer="91"/>
+<label x="33.02" y="152.4" size="1.778" layer="95"/>
+</segment>
+<segment>
+<pinref part="C10" gate="G$1" pin="2"/>
+<wire x1="289.56" y1="180.34" x2="292.1" y2="180.34" width="0.1524" layer="91"/>
+<wire x1="292.1" y1="180.34" x2="292.1" y2="170.18" width="0.1524" layer="91"/>
+<pinref part="C9" gate="G$1" pin="2"/>
+<wire x1="292.1" y1="170.18" x2="292.1" y2="167.64" width="0.1524" layer="91"/>
+<wire x1="289.56" y1="170.18" x2="292.1" y2="170.18" width="0.1524" layer="91"/>
+<junction x="292.1" y="170.18"/>
+<pinref part="GND6" gate="1" pin="GND"/>
 </segment>
 </net>
@@
 <pinref part="+3V5" gate="G$1" pin="+3V3"/>
 </segment>
+<segment>
+<pinref part="ICSP" gate="G$1" pin="4"/>
+<wire x1="27.94" y1="154.94" x2="40.64" y2="154.94" width="0.1524" layer="91"/>
+<label x="33.02" y="154.94" size="1.778" layer="95"/>
+</segment>
 </net>
 <net name="MCLR" class="0">
@@
 <pinref part="R1" gate="G$1" pin="2"/>
 <label x="96.52" y="175.26" size="1.778" layer="95"/>
+</segment>
+<segment>
+<pinref part="ICSP" gate="G$1" pin="1"/>
+<wire x1="27.94" y1="162.56" x2="40.64" y2="162.56" width="0.1524" layer="91"/>
+<label x="33.02" y="162.56" size="1.778" layer="95"/>
 </segment>
 </net>
@@
 </segment>
 </net>
+<net name="PGEC1" class="0">
+<segment>
+<pinref part="ICSP" gate="G$1" pin="2"/>
+<wire x1="27.94" y1="160.02" x2="40.64" y2="160.02" width="0.1524" layer="91"/>
+<label x="33.02" y="160.02" size="1.778" layer="95"/>
+</segment>
+<segment>
+<pinref part="U1" gate="G$1" pin="PGEC1/OA1IN+/AN4/C1IN1+/C1IN3-/C2IN3-/RPB2/RB2"/>
+<wire x1="114.3" y1="142.24" x2="93.98" y2="142.24" width="0.1524" layer="91"/>
+<label x="93.98" y="142.24" size="1.778" layer="95"/>
+</segment>
+</net>
+<net name="PGED1" class="0">
+<segment>
+<pinref part="ICSP" gate="G$1" pin="3"/>
+<wire x1="27.94" y1="157.48" x2="40.64" y2="157.48" width="0.1524" layer="91"/>
+<label x="33.02" y="157.48" size="1.778" layer="95"/>
+</segment>
+<segment>
+<pinref part="U1" gate="G$1" pin="PGED1/OA1IN-/AN5/CTCMP/C1IN1-/RTCC/RPB3/RB3"/>
+<wire x1="114.3" y1="139.7" x2="93.98" y2="139.7" width="0.1524" layer="91"/>
+<label x="93.98" y="139.7" size="1.778" layer="95"/>
+</segment>
+</net>
+<net name="NC1" class="0">
+<segment>
+<pinref part="ICSP" gate="G$1" pin="6"/>
+<wire x1="27.94" y1="149.86" x2="40.64" y2="149.86" width="0.1524" layer="91"/>
+<label x="33.02" y="149.86" size="1.778" layer="95"/>
+</segment>
+</net>
+<net name="OSCIN" class="0">
+<segment>
+<pinref part="U1" gate="G$1" pin="OSCI/CLKI/AN49/CVD49/RPC12/RC12"/>
+<wire x1="254" y1="175.26" x2="274.32" y2="175.26" width="0.1524" layer="91"/>
+<pinref part="C10" gate="G$1" pin="1"/>
+<wire x1="274.32" y1="175.26" x2="274.32" y2="180.34" width="0.1524" layer="91"/>
+<wire x1="274.32" y1="180.34" x2="279.4" y2="180.34" width="0.1524" layer="91"/>
+<pinref part="Q1" gate="G$1" pin="1"/>
+<wire x1="279.4" y1="180.34" x2="281.94" y2="180.34" width="0.1524" layer="91"/>
+<wire x1="279.4" y1="177.8" x2="279.4" y2="180.34" width="0.1524" layer="91"/>
+<junction x="279.4" y="180.34"/>
+</segment>
+</net>
+<net name="OSCOUT" class="0">
+<segment>
+<pinref part="U1" gate="G$1" pin="OSCO/CLKO/RPC15/RC15"/>
+<wire x1="254" y1="172.72" x2="274.32" y2="172.72" width="0.1524" layer="91"/>
+<pinref part="C9" gate="G$1" pin="1"/>
+<wire x1="274.32" y1="172.72" x2="274.32" y2="170.18" width="0.1524" layer="91"/>
+<wire x1="274.32" y1="170.18" x2="279.4" y2="170.18" width="0.1524" layer="91"/>
+<pinref part="Q1" gate="G$1" pin="2"/>
+<wire x1="279.4" y1="170.18" x2="281.94" y2="170.18" width="0.1524" layer="91"/>
+<wire x1="279.4" y1="172.72" x2="279.4" y2="170.18" width="0.1524" layer="91"/>
+<junction x="279.4" y="170.18"/>
+</segment>
+</net>
