File: 80%/rev0.1.sch (EAGLE design)
At the start: 11 parts, among them U1 PIC32MK1024MCF100100TQFP

Commit message: added keys!!!
Parts:
- added C10, C11, C9: 0.1uF, resistor:C-USC0603
- added J1, J2: USB-B, SparkFun-Connectors:USBPTH
- added JP1: (no value), adafruit:PINHD-1X6LOCK
- added Q1: (no value), adafruit:CRYSTALCTS406
- added SW1, SW10, SW11, SW12, SW13, SW14, SW15, SW16, SW17, SW18, SW19, SW2, SW20, SW21, SW22, SW23, SW24, SW25, SW26, SW27, SW28, SW29, SW3, SW30, SW31, SW32, SW33, SW34, SW35, SW36, SW37, SW38, SW39, SW4, SW40, SW41, SW42, SW43, SW44, SW45, SW46, SW47, SW48, SW49, SW5, SW50, SW51, SW52, SW53, SW54, SW55, SW56, SW57, SW58, SW59, SW6, SW60, SW61, SW62, SW63, SW64, SW65, SW66, SW67, SW68, SW69, SW7, SW70, SW71, SW72, SW73, SW74, SW75, SW76, SW77, SW78, SW79, SW8, SW80, SW81, SW82, SW83, SW84, SW85, SW86, SW87, SW88, SW89, SW9, SW90, SW91, SW92: CHERRY_MX, ALLEYBEACH_LIB:CHERRY_MX
- C1, C2, C3, C4, C5, C6: device resistor:C-USC0805 -> resistor:C-USC0603
- C7: value 47uF -> 0.1uF; device resistor:C-USC0805 -> resistor:C-USC0603
- C8: value 4.7uF -> 0.1uF; device resistor:C-USC0805 -> resistor:C-USC0603
- R1, R2: device resistor:R-US_R0805 -> resistor:R-US_R0603
Connections:
- removed net +3V3: C1.1, C2.1, C3.1, C4.1, C5.1, C7.1, C8.1, R2.2, U1.VBUS3V3, U1.VDD@16, U1.VDD@2, U1.VDD@37, U1.VDD@46, U1.VDD@62, U1.VDD@86
- new net N$1: C7.1, U1.AVDD
- new net N$2: C7.2, U1.AVSS
- new net N$3: C8.1, R1.1, R2.1
- new net N$4: C9.1, Q1.2, U1.OSCI/CLKI/AN49/CVD49/RPC12/RC12
- new net PGEC1: JP1.2, U1.PGEC1/OA1IN+/AN4/C1IN1+/C1IN3-/C2IN3-/RPB2/RB2
- new net PGED1: JP1.3, U1.PGED1/OA1IN-/AN5/CTCMP/C1IN1-/RTCC/RPB3/RB3
- new net USB1_N: J1.D-, U1.D1-
- new net USB1_P: J1.D+, U1.D1+
- new net USB2_N: J2.D-, U1.D2-
- new net USB2_P: J2.D+, U1.D2+
- new net VBUS1: J1.VBUS, U1.VBUS
- new net VBUS2: J2.VBUS, U1.VBUS2
- new net VCC3V3: C1.1, C11.1, C2.1, C3.1, C4.1, C5.1, C6.1, JP1.4, R2.2, U1.VBUS3V3, U1.VDD@16, U1.VDD@2, U1.VDD@37, U1.VDD@46, U1.VDD@62, U1.VDD@86
- net GND: now also C10.2, C11.2, C9.2, J1.GND@2, J2.GND@2, JP1.5; no longer C7.2
- net MCLR: now also JP1.1
- net N$5: now also C10.1, Q1.1, U1.OSCO/CLKO/RPC15/RC15; no longer C6.1, R1.1, R2.1
Other:
- note removed: "9 keys"
- note removed: "?"
- note removed: "Block Diagram"
- note removed: "Buck/ Boost"
- note removed: "LCD"
- note removed: "LDO"
- note removed: "MCU"
- note removed: "add decoupling cap to each pin"
- note removed: "usb"
- moved on the sheet: C1, C2, C3, C4, C5, C6, C7, C8, R1, R2, U1

Commit message: laying matrix done
laying matrix done
Parts:
- removed SW85: CHERRY_MX, ALLEYBEACH_LIB:CHERRY_MX
- added CAPS, LED1\, SCROLL: (no value), adafruit:LEDCHIP-LED0805
- added D1, D10, D11, D12, D13, D14, D15, D16, D17, D18, D19, D2, D20, D21, D22, D23, D24, D25, D26, D27, D28, D29, D3, D30, D31, D32, D33, D34, D35, D36, D37, D38, D39, D4, D40, D41, D42, D43, D44, D45, D46, D47, D48, D49, D5, D50, D51, D52, D53, D54, D55, D56, D57, D58, D59, D6, D60, D61, D62, D63, D64, D65, D66, D67, D68, D69, D7, D70, D71, D72, D73, D74, D75, D76, D77, D78, D79, D8, D80, D81, D82, D83, D84, D85, D86, D87, D88, D89, D9, D90, D91, D92: (no value), adafruit:DIODESOD-123
- added SPACE: CHERRY_MX, ALLEYBEACH_LIB:CHERRY_MX
Connections:
- new net C1: SW1.1, SW18.1, SW36.1, SW54.1, SW68.1, SW82.1
- new net C2: SW19.1, SW2.1, SW37.1, SW55.1, SW69.1, SW83.1
- new net C3: SW20.1, SW3.1, SW38.1, SW56.1, SW70.1, SW84.1
- new net C4: SPACE.1, SW21.1, SW39.1, SW4.1, SW57.1, SW71.1
- new net C5: SW22.1, SW40.1, SW5.1, SW58.1, SW72.1, SW86.1
- new net C6: SW23.1, SW41.1, SW59.1, SW6.1, SW73.1, SW87.1
- new net N$10: D3.A, SW36.2
- new net N$100: D50.A, SW26.2
- new net N$101: D44.A, SW25.2
- new net N$102: D43.A, SW8.2
- new net N$103: D49.A, SW9.2
- new net N$104: D37.A, SW7.2
- new net N$105: D38.A, SW24.2
- new net N$106: D39.A, SW42.2
- new net N$107: D40.A, SW60.2
- new net N$108: D41.A, SW74.2
- new net N$109: D42.A, SW88.2
- new net N$11: D2.A, SW18.2
- new net N$12: D1.A, SW1.2
- new net N$13: D91.A, SW35.2
- new net N$14: D7.A, SW2.2
- new net N$15: D12.A, SW83.2
- new net N$16: D11.A, SW69.2
- new net N$17: D10.A, SW55.2
- new net N$18: D9.A, SW37.2
- new net N$19: D8.A, SW19.2
- new net N$20: D92.A, SW53.2
- new net N$21: D90.A, SW52.2
- new net N$22: D89.A, SW34.2
- new net N$23: D85.A, SW16.2
- new net N$24: SW24.1, SW42.1, SW60.1, SW7.1, SW74.1, SW88.1
- new net N$25: SW25.1, SW43.1, SW61.1, SW75.1, SW8.1, SW89.1
- new net N$26: SW44.1, SW62.1, SW76.1, SW9.1, SW90.1
- new net N$27: SW10.1, SW27.1, SW45.1, SW63.1, SW77.1, SW91.1
- new net N$28: SW11.1, SW28.1, SW46.1, SW64.1, SW78.1, SW92.1
- new net N$29: SW12.1, SW29.1, SW47.1, SW65.1, SW79.1
- new net N$30: SW13.1, SW30.1, SW48.1, SW66.1, SW80.1
- new net N$31: SW14.1, SW31.1, SW49.1, SW67.1, SW81.1
- new net N$32: SW15.1, SW32.1, SW50.1
- new net N$33: SW16.1, SW33.1, SW51.1
- new net N$34: SW17.1, SW34.1, SW52.1
- new net N$35: SW35.1, SW53.1
- new net N$36: D14.A, SW20.2
- new net N$37: D13.A, SW3.2
- new net N$38: D15.A, SW38.2
- new net N$39: D21.A, SW39.2
- new net N$40: D20.A, SW21.2
- new net N$41: D22.A, SW57.2
- new net N$42: D16.A, SW56.2
- new net N$43: D17.A, SW70.2
- new net N$44: D23.A, SW71.2
- new net N$45: D24.A, SPACE.2
- new net N$46: D18.A, SW84.2
- new net N$47: D19.A, SW4.2
- new net N$48: D25.A, SW5.2
- new net N$49: D31.A, SW6.2
- new net N$50: D26.A, SW22.2
- new net N$51: D32.A, SW23.2
- new net N$52: D33.A, SW41.2
- new net N$53: D27.A, SW40.2
- new net N$54: D28.A, SW58.2
- new net N$55: D34.A, SW59.2
- new net N$56: D35.A, SW73.2
- new net N$57: D29.A, SW72.2
- new net N$58: D30.A, SW86.2
- new net N$59: D36.A, SW87.2
- new net N$6: D88.A, SW17.2
- new net N$60: D86.A, SW33.2
- new net N$61: D87.A, SW51.2
- new net N$62: D84.A, SW50.2
- new net N$63: D83.A, SW32.2
- new net N$64: D82.A, SW15.2
- new net N$65: D77.A, SW14.2
- new net N$66: D78.A, SW31.2
- new net N$67: D79.A, SW49.2
- new net N$68: D80.A, SW67.2
- new net N$69: D81.A, SW81.2
- new net N$7: D6.A, SW82.2
- new net N$70: D76.A, SW80.2
- new net N$71: D75.A, SW66.2
- new net N$72: D70.A, SW65.2
- new net N$73: D71.A, SW79.2
- new net N$74: D69.A, SW47.2
- new net N$75: D74.A, SW48.2
- new net N$76: D73.A, SW30.2
- new net N$77: D68.A, SW29.2
- new net N$78: D67.A, SW12.2
- new net N$79: D72.A, SW13.2
- new net N$8: D5.A, SW68.2
- new net N$80: D61.A, SW11.2
- new net N$81: D55.A, SW10.2
- new net N$82: D56.A, SW27.2
- new net N$83: D62.A, SW28.2
- new net N$84: D63.A, SW46.2
- new net N$85: D57.A, SW45.2
- new net N$86: D58.A, SW63.2
- new net N$87: D64.A, SW64.2
- new net N$88: D65.A, SW78.2
- new net N$89: D59.A, SW77.2
- new net N$9: D4.A, SW54.2
- new net N$90: D60.A, SW91.2
- new net N$91: D66.A, SW92.2
- new net N$92: D48.A, SW89.2
- new net N$93: D54.A, SW90.2
- new net N$94: D47.A, SW75.2
- new net N$95: D53.A, SW76.2
- new net N$96: D52.A, SW62.2
- new net N$97: D46.A, SW61.2
- new net N$98: D45.A, SW43.2
- new net N$99: D51.A, SW44.2
- new net R1: D1.C, D13.C, D19.C, D25.C, D31.C, D37.C, D43.C, D49.C, D55.C, D61.C, D67.C, D7.C, D72.C, D77.C, D82.C, D85.C, D88.C
- new net R2: D14.C, D2.C, D20.C, D26.C, D32.C, D38.C, D44.C, D50.C, D56.C, D62.C, D68.C, D73.C, D78.C, D8.C, D83.C, D86.C, D89.C, D91.C
- new net R3: D15.C, D21.C, D27.C, D3.C, D33.C, D39.C, D45.C, D51.C, D57.C, D63.C, D69.C, D74.C, D79.C, D84.C, D87.C, D9.C, D90.C, D92.C
- new net R4: D10.C, D16.C, D22.C, D28.C, D34.C, D4.C, D40.C, D46.C, D52.C, D58.C, D64.C, D70.C, D75.C, D80.C
- new net R5: D11.C, D17.C, D23.C, D29.C, D35.C, D41.C, D47.C, D5.C, D53.C, D59.C, D65.C, D71.C, D76.C, D81.C
- new net R6: D12.C, D18.C, D24.C, D30.C, D36.C, D42.C, D48.C, D54.C, D6.C, D60.C, D66.C
Other:
- moved on the sheet: SW1, SW10, SW11, SW12, SW13, SW14, SW15, SW16, SW17, SW18, SW19, SW2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
