File: 80%/rev0.1.brd (EAGLE design)
At the start: 375.5 x 123.8 mm, 208 parts, among them J1 USB-B, Q1 48MHz, SW1 CHERRY_MX, SW10 CHERRY_MX, SW11 CHERRY_MX, SW12 CHERRY_MX, SW13 CHERRY_MX, SW14 CHERRY_MX, SW15 CHERRY_MX, SW16 CHERRY_MX, SW17 CHERRY_MX, SW18 CHERRY_MX, SW19 CHERRY_MX, SW2 CHERRY_MX, SW20 CHERRY_MX, SW21 CHERRY_MX, SW22 CHERRY_MX, SW23 CHERRY_MX, SW24 CHERRY_MX, SW25 CHERRY_MX, SW26 CHERRY_MX, SW27 CHERRY_MX, SW28 CHERRY_MX, SW29 CHERRY_MX, SW3 CHERRY_MX, SW30 CHERRY_MX, SW31 CHERRY_MX, SW32 CHERRY_MX, SW33 CHERRY_MX, SW34 CHERRY_MX, SW35 CHERRY_MX, SW36 CHERRY_MX, SW37 CHERRY_MX, SW38 CHERRY_MX, SW39 CHERRY_MX, SW4 CHERRY_MX, SW40 CHERRY_MX, SW41 CHERRY_MX, SW42 CHERRY_MX, SW43 CHERRY_MX, SW44 CHERRY_MX, SW45 CHERRY_MX, SW46 CHERRY_MX, SW47 CHERRY_MX, SW48 CHERRY_MX, SW49 CHERRY_MX, SW5 CHERRY_MX, SW50 CHERRY_MX, SW51 CHERRY_MX, SW52 CHERRY_MX, SW53 CHERRY_MX, SW54 CHERRY_MX, SW55 CHERRY_MX, SW56 CHERRY_MX, SW57 CHERRY_MX, SW58 CHERRY_MX, SW59 CHERRY_MX, SW6 CHERRY_MX, SW60 CHERRY_MX, SW61 CHERRY_MX, SW62 CHERRY_MX, SW63 CHERRY_MX, SW64 CHERRY_MX, SW65 CHERRY_MX, SW66 CHERRY_MX, SW67 CHERRY_MX, SW68 CHERRY_MX, SW69 CHERRY_MX, SW7 CHERRY_MX, SW70 CHERRY_MX, SW71 CHERRY_MX, SW72 CHERRY_MX, SW73 CHERRY_MX, SW74 CHERRY_MX, SW75 CHERRY_MX, SW76 CHERRY_MX, SW77 CHERRY_MX, SW78 CHERRY_MX, SW79 CHERRY_MX, SW8 CHERRY_MX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

Commit message: closer to clean
Parts:
- moved C1 124.0 mm to (503.9, 75.7)
- moved C2 120.8 mm to (503.9, 81.5)
- moved C3 117.7 mm to (503.9, 87.4)
- moved C5 106.2 mm to (503.9, 100.1)
- moved C6 106.2 mm to (503.9, 106.4)
- moved C4 106.2 mm to (503.9, 93.7)
- moved C7 95.6 mm to (503.9, 112.8)
- moved C12 80.7 mm to (503.9, 144.5)
- moved C8 78.4 mm to (503.9, 119.1), turned to 180 degrees
- moved C9 74.9 mm to (503.9, 125.5), turned to 180 degrees
- moved C10 68.9 mm to (503.9, 131.8), turned to 180 degrees
- moved C11 66.4 mm to (503.9, 138.2), turned to 180 degrees
- moved TP1 60.0 mm to (501.6, 157.2)
- moved C13 55.8 mm to (503.9, 162.3), turned to 180 degrees
- moved SJ1 39.9 mm to (475.0, 153.7)
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Routing:
- net RESET: track 65.5 -> 0.00 mm
- net SWCLK: track 61.0 -> 0.00 mm
- net SWDIO: track 48.9 -> 0.00 mm
- net SWO: track 32.2 -> 0.00 mm
- net VCC3V3: track 27.8 -> 0.00 mm
- net N$2: track 17.6 -> 0.00 mm
- net VBUS1: track 14.0 -> 0.00 mm
- net USB1_P: track 22.1 -> 15.3 mm
- net USB1_N: track 21.6 -> 15.1 mm
