File: 80%/rev0.1 parts placement.brd (EAGLE design)
At the start: 375.5 x 123.8 mm, 217 parts, among them J1 USB-B, Q1 48MHz, SW1 CHERRY_MX, SW10 CHERRY_MX, SW11 CHERRY_MX, SW12 CHERRY_MX, SW13 CHERRY_MX, SW14 CHERRY_MX, SW15 CHERRY_MX, SW16 CHERRY_MX, SW17 CHERRY_MX, SW18 CHERRY_MX, SW19 CHERRY_MX, SW2 CHERRY_MX, SW20 CHERRY_MX, SW21 CHERRY_MX, SW22 CHERRY_MX, SW23 CHERRY_MX, SW24 CHERRY_MX, SW25 CHERRY_MX, SW26 CHERRY_MX, SW27 CHERRY_MX, SW28 CHERRY_MX, SW29 CHERRY_MX, SW3 CHERRY_MX, SW30 CHERRY_MX, SW31 CHERRY_MX, SW32 CHERRY_MX, SW33 CHERRY_MX, SW34 CHERRY_MX, SW35 CHERRY_MX, SW36 CHERRY_MX, SW37 CHERRY_MX, SW38 CHERRY_MX, SW39 CHERRY_MX, SW4 CHERRY_MX, SW40 CHERRY_MX, SW41 CHERRY_MX, SW42 CHERRY_MX, SW43 CHERRY_MX, SW44 CHERRY_MX, SW45 CHERRY_MX, SW46 CHERRY_MX, SW47 CHERRY_MX, SW48 CHERRY_MX, SW49 CHERRY_MX, SW5 CHERRY_MX, SW50 CHERRY_MX, SW51 CHERRY_MX, SW52 CHERRY_MX, SW53 CHERRY_MX, SW54 CHERRY_MX, SW55 CHERRY_MX, SW56 CHERRY_MX, SW57 CHERRY_MX, SW58 CHERRY_MX, SW59 CHERRY_MX, SW6 CHERRY_MX, SW60 CHERRY_MX, SW61 CHERRY_MX, SW62 CHERRY_MX, SW63 CHERRY_MX, SW64 CHERRY_MX, SW65 CHERRY_MX, SW66 CHERRY_MX, SW67 CHERRY_MX, SW68 CHERRY_MX, SW69 CHERRY_MX, SW7 CHERRY_MX, SW70 CHERRY_MX, SW71 CHERRY_MX, SW72 CHERRY_MX, SW73 CHERRY_MX, SW74 CHERRY_MX, SW75 CHERRY_MX, SW76 CHERRY_MX, SW77 CHERRY_MX, SW78 CHERRY_MX, SW79 CHERRY_MX, SW8 CHERRY_MX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

Commit message: cleaned up a little
added power routing
Parts:
- added C16: 4.7uF, resistor:C0805
- added C17: 33nF, resistor:C0402
- added C18: 2.2uF, resistor:C0805
- added R6: 100K, resistor:R0402
- added U2: LP3982IMM-3.3/NOPB, clackboard_lib:LP3982IMM-3.3/NOPB
- moved C4 44.1 mm to (276.9, 34.3), flipped to the bottom, turned to 0 degrees
- moved C5 39.6 mm to (277.4, 32.5), flipped to the bottom, turned to 0 degrees
- moved C6 36.6 mm to (277.4, 31.2), flipped to the bottom, turned to 0 degrees
Connections:
- new net N$31: C17.1, U2.6
- new net N$32: R6.1, U2.8
- net GND: now also C16.2, C17.2, C18.2, U2.3
- net VBUS1: now also C16.1, U2.2, U2.7
- net VCC3V3: now also C18.1, R6.2, U2.1, U2.4
Routing:
- net VBUS1: track 72.7 -> 143.4 mm, vias 2 -> 4
- net VCC3V3: track 161.6 -> 211.4 mm, vias 6 -> 8
- net GND: track 206.8 -> 194.0 mm, vias 8 -> 86
- net N$32: track 0.00 -> 2.06 mm
- net N$31: track 0.00 -> 2.04 mm
- net R4: track 460.7 -> 458.9 mm
- net C13: track 217.0 -> 217.8 mm
- net C14: vias 1 -> 2
Other:
- board text added: "Hardware: Scott Griffitts"
- board text added: "Software: Andrew Kurtz"

Commit message: update
Routing:
- net GND: vias 86 -> 97
Changed lines of the file:
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@@
 <?xml version="1.0" encoding="utf-8"?>
 <!DOCTYPE eagle SYSTEM "eagle.dtd">
-<eagle version="8.3.1">
+<eagle version="8.4.3">
 <drawing>
 <settings>
@@
 <param name="dpMaxLengthDifference" value="10mm"/>
 <param name="dpGapFactor" value="1"/>
-<param name="checkGrid" value="0"/>
 <param name="checkAngle" value="0"/>
 <param name="checkFont" value="1"/>
 <param name="checkRestrict" value="1"/>
+<param name="checkStop" value="0"/>
 <param name="useDiameter" value="13"/>
 <param name="maxErrors" value="50"/>
@@
 <via x="12.192" y="26.67" extent="1-16" drill="0.3"/>
 <via x="107.442" y="69.088" extent="1-16" drill="0.3"/>
+<via x="345.741" y="121.8475" extent="1-16" drill="0.3"/>
+<via x="357.425" y="121.8475" extent="1-16" drill="0.3"/>
+<via x="350.313" y="96.4475" extent="1-16" drill="0.3"/>
+<via x="284.781" y="94.1615" extent="1-16" drill="0.3"/>
+<via x="282.749" y="94.1615" extent="1-16" drill="0.3"/>
+<via x="282.749" y="87.8115" extent="1-16" drill="0.3"/>
+<via x="284.781" y="87.8115" extent="1-16" drill="0.3"/>
+<via x="282.749" y="81.7155" extent="1-16" drill="0.3"/>
+<via x="284.781" y="81.7155" extent="1-16" drill="0.3"/>
+<via x="282.702" y="71.374" extent="1-16" drill="0.3"/>
+<via x="284.734" y="71.374" extent="1-16" drill="0.3"/>
 </signal>
 <signal name="USB1_N">
@@
 <wire x1="366.844371875" y1="40" x2="366.136" y2="40" width="0.1524" layer="16"/>
 <wire x1="366.844371875" y1="40" x2="366.85" y2="40" width="0.1524" layer="16"/>
-<wire x1="21.85" y1="40" x2="27.564" y2="40" width="0.6096" layer="16"/>
+<wire x1="27.564" y1="40" x2="21.85" y2="40" width="0.6096" layer="16"/>
 <wire x1="27.564" y1="40" x2="28.956" y2="38.608" width="0.6096" layer="16"/>
 <wire x1="216.8742125" y1="38.608" x2="236.838825" y2="38.608" width="0.6096" layer="16"/>
