File: 80%/rev0.1 parts placement.brd (EAGLE design)
At the start: 375.5 x 123.8 mm, 222 parts, among them J1 USB-B, Q1 48MHz, SW1 CHERRY_MX, SW10 CHERRY_MX, SW11 CHERRY_MX, SW12 CHERRY_MX, SW13 CHERRY_MX, SW14 CHERRY_MX, SW15 CHERRY_MX, SW16 CHERRY_MX, SW17 CHERRY_MX, SW18 CHERRY_MX, SW19 CHERRY_MX, SW2 CHERRY_MX, SW20 CHERRY_MX, SW21 CHERRY_MX, SW22 CHERRY_MX, SW23 CHERRY_MX, SW24 CHERRY_MX, SW25 CHERRY_MX, SW26 CHERRY_MX, SW27 CHERRY_MX, SW28 CHERRY_MX, SW29 CHERRY_MX, SW3 CHERRY_MX, SW30 CHERRY_MX, SW31 CHERRY_MX, SW32 CHERRY_MX, SW33 CHERRY_MX, SW34 CHERRY_MX, SW35 CHERRY_MX, SW36 CHERRY_MX, SW37 CHERRY_MX, SW38 CHERRY_MX, SW39 CHERRY_MX, SW4 CHERRY_MX, SW40 CHERRY_MX, SW41 CHERRY_MX, SW42 CHERRY_MX, SW43 CHERRY_MX, SW44 CHERRY_MX, SW45 CHERRY_MX, SW46 CHERRY_MX, SW47 CHERRY_MX, SW48 CHERRY_MX, SW49 CHERRY_MX, SW5 CHERRY_MX, SW50 CHERRY_MX, SW51 CHERRY_MX, SW52 CHERRY_MX, SW53 CHERRY_MX, SW54 CHERRY_MX, SW55 CHERRY_MX, SW56 CHERRY_MX, SW57 CHERRY_MX, SW58 CHERRY_MX, SW59 CHERRY_MX, SW6 CHERRY_MX, SW60 CHERRY_MX, SW61 CHERRY_MX, SW62 CHERRY_MX, SW63 CHERRY_MX, SW64 CHERRY_MX, SW65 CHERRY_MX, SW66 CHERRY_MX, SW67 CHERRY_MX, SW68 CHERRY_MX, SW69 CHERRY_MX, SW7 CHERRY_MX, SW70 CHERRY_MX, SW71 CHERRY_MX, SW72 CHERRY_MX, SW73 CHERRY_MX, SW74 CHERRY_MX, SW75 CHERRY_MX, SW76 CHERRY_MX, SW77 CHERRY_MX, SW78 CHERRY_MX, SW79 CHERRY_MX, SW8 CHERRY_MX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

Commit message: 80 update
updated the 80% with a new diode.
Parts:
- added TP10, TP11, TP12, TP13, TP14, TP15, TP16, TP17, TP18, TP3, TP4, TP5, TP6, TP7, TP8, TP9: PTR1B1,27, testpad:B1,27
- D1, D10, D11, D12, D13, D14, D15, D16, D17, D18, D19, D2, D20, D21, D22, D23, D24, D25, D26, D27, D28, D29, D3, D30, D31, D32, D33, D34, D35, D36, D37, D38, D39, D4, D40, D41, D42, D43, D44, D45, D46, D47, D48, D49, D5, D50, D51, D52, D53, D54, D55, D56, D57, D58, D59, D6, D60, D61, D62, D63, D64, D65, D66, D67, D68, D69, D7, D70, D71, D72, D73, D74, D75, D76, D77, D78, D79, D8, D80, D81, D82, D83, D84, D85, D86, D87, D88, D89, D9, D90, D91, D92: value (none) -> 1N4148; device adafruit:SOD-123 -> clackboard_lib:SOD323
- moved D5 7.28 mm to (23.0, 22.0)
- moved D6 7.28 mm to (13.0, 3.00)
- moved D20 7.07 mm to (68.0, 79.0)
- moved D50 7.07 mm to (163.0, 79.0)
- moved D14 6.08 mm to (49.0, 79.0)
- moved D44 6.08 mm to (144.0, 79.0)
- moved D73 6.08 mm to (239.0, 79.0)
- moved D89 6.08 mm to (339.0, 79.0)
- moved D35 5.39 mm to (130.0, 22.0)
- moved D34 5.10 mm to (120.0, 41.0)
- moved D38 5.10 mm to (125.0, 79.0)
- moved D68 5.10 mm to (220.0, 79.0)
- moved D8 5.10 mm to (30.0, 79.0)
- moved D86 5.10 mm to (320.0, 79.0)
- moved D12 5.00 mm to (40.0, 5.00)
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Connections:
- new net N$110: TP12.TP, U1.30
- new net N$111: TP11.TP, U1.31
- new net N$112: TP10.TP, U1.32
- new net N$113: TP9.TP, U1.36
- new net N$114: TP8.TP, U1.37
- new net N$115: TP7.TP, U1.38
- new net N$116: TP5.TP, U1.41
- new net N$117: TP4.TP, U1.42
- new net N$118: TP3.TP, U1.43
- new net N$119: TP17.TP, U1.53
- new net N$120: TP18.TP, U1.54
- new net N$30: TP16.TP, U1.19
- new net N$33: TP15.TP, U1.21
- new net N$34: TP14.TP, U1.28
- new net N$35: TP13.TP, U1.29
- net N$10: now also D3.2; no longer D3.A
- net N$100: now also D50.2; no longer D50.A
- net N$101: now also D44.2; no longer D44.A
- net N$102: now also D43.2; no longer D43.A
- net N$103: now also D49.2; no longer D49.A
- net N$104: now also D37.2; no longer D37.A
- net N$105: now also D38.2; no longer D38.A
- net N$106: now also D39.2; no longer D39.A
- net N$107: now also D40.2; no longer D40.A
- net N$108: now also D41.2; no longer D41.A
- net N$109: now also D42.2; no longer D42.A
- net N$11: now also D2.2; no longer D2.A
- net N$12: now also D1.2; no longer D1.A
- net N$13: now also D91.2; no longer D91.A
- net N$14: now also D7.2; no longer D7.A
- net N$15: now also D12.2; no longer D12.A
- net N$16: now also D11.2; no longer D11.A
- net N$17: now also D10.2; no longer D10.A
- net N$18: now also D9.2; no longer D9.A
- net N$19: now also D8.2; no longer D8.A
- net N$20: now also D92.2; no longer D92.A
- net N$21: now also D90.2; no longer D90.A
- net N$22: now also D89.2; no longer D89.A
- net N$23: now also D85.2; no longer D85.A
- net N$36: now also D14.2; no longer D14.A
- net N$37: now also D13.2; no longer D13.A
- net N$38: now also D15.2; no longer D15.A
- net N$39: now also D21.2; no longer D21.A
- net N$40: now also D20.2; no longer D20.A
- net N$41: now also D22.2; no longer D22.A
- net N$42: now also D16.2; no longer D16.A
- net N$43: now also D17.2; no longer D17.A
- net N$44: now also D23.2; no longer D23.A
- net N$45: now also D24.2; no longer D24.A
- net N$46: now also D18.2; no longer D18.A
- net N$47: now also D19.2; no longer D19.A
- net N$48: now also D25.2; no longer D25.A
- net N$49: now also D31.2; no longer D31.A
- net N$50: now also D26.2; no longer D26.A
- net N$51: now also D32.2; no longer D32.A
- net N$52: now also D33.2; no longer D33.A
- net N$53: now also D27.2; no longer D27.A
- net N$54: now also D28.2; no longer D28.A
- net N$55: now also D34.2; no longer D34.A
- net N$56: now also D35.2; no longer D35.A
- net N$57: now also D29.2; no longer D29.A
- net N$58: now also D30.2; no longer D30.A
- net N$59: now also D36.2; no longer D36.A
- net N$6: now also D88.2; no longer D88.A
- net N$60: now also D86.2; no longer D86.A
- net N$61: now also D87.2; no longer D87.A
- net N$62: now also D84.2; no longer D84.A
- net N$63: now also D83.2; no longer D83.A
- net N$64: now also D82.2; no longer D82.A
- net N$65: now also D77.2; no longer D77.A
- net N$66: now also D78.2; no longer D78.A
- net N$67: now also D79.2; no longer D79.A
- net N$68: now also D80.2; no longer D80.A
- net N$69: now also D81.2; no longer D81.A
- net N$7: now also D6.2; no longer D6.A
- net N$70: now also D76.2; no longer D76.A
- net N$71: now also D75.2; no longer D75.A
- net N$72: now also D70.2; no longer D70.A
- net N$73: now also D71.2; no longer D71.A
- net N$74: now also D69.2; no longer D69.A
- net N$75: now also D74.2; no longer D74.A
- net N$76: now also D73.2; no longer D73.A
- net N$77: now also D68.2; no longer D68.A
- net N$78: now also D67.2; no longer D67.A
- net N$79: now also D72.2; no longer D72.A
- net N$8: now also D5.2; no longer D5.A
- net N$80: now also D61.2; no longer D61.A
- net N$81: now also D55.2; no longer D55.A
- net N$82: now also D56.2; no longer D56.A
- net N$83: now also D62.2; no longer D62.A
- net N$84: now also D63.2; no longer D63.A
- net N$85: now also D57.2; no longer D57.A
- net N$86: now also D58.2; no longer D58.A
- net N$87: now also D64.2; no longer D64.A
- net N$88: now also D65.2; no longer D65.A
- net N$89: now also D59.2; no longer D59.A
- net N$9: now also D4.2; no longer D4.A
- net N$90: now also D60.2; no longer D60.A
- net N$91: now also D66.2; no longer D66.A
- net N$92: now also D48.2; no longer D48.A
- net N$93: now also D54.2; no longer D54.A
- net N$94: now also D47.2; no longer D47.A
- net N$95: now also D53.2; no longer D53.A
- net N$96: now also D52.2; no longer D52.A
- net N$97: now also D46.2; no longer D46.A
- net N$98: now also D45.2; no longer D45.A
- net N$99: now also D51.2; no longer D51.A
- net R1: now also D1.1, D13.1, D19.1, D25.1, D31.1, D37.1, D43.1, D49.1, D55.1, D61.1, D67.1, D7.1, D72.1, D77.1, D82.1, D85.1, D88.1; no longer D1.C, D13.C, D19.C, D25.C, D31.C, D37.C, D43.C, D49.C, D55.C, D61.C, D67.C, D7.C, D72.C, D77.C, D82.C, D85.C, D88.C
- net R2: now also D14.1, D2.1, D20.1, D26.1, D32.1, D38.1, D44.1, D50.1, D56.1, D62.1, D68.1, D73.1, D78.1, D8.1, D83.1, D86.1, D89.1, D91.1; no longer D14.C, D2.C, D20.C, D26.C, D32.C, D38.C, D44.C, D50.C, D56.C, D62.C, D68.C, D73.C, D78.C, D8.C, D83.C, D86.C, D89.C, D91.C
- net R3: now also D15.1, D21.1, D27.1, D3.1, D33.1, D39.1, D45.1, D51.1, D57.1, D63.1, D69.1, D74.1, D79.1, D84.1, D87.1, D9.1, D90.1, D92.1; no longer D15.C, D21.C, D27.C, D3.C, D33.C, D39.C, D45.C, D51.C, D57.C, D63.C, D69.C, D74.C, D79.C, D84.C, D87.C, D9.C, D90.C, D92.C
- net R4: now also D10.1, D16.1, D22.1, D28.1, D34.1, D4.1, D40.1, D46.1, D52.1, D58.1, D64.1, D70.1, D75.1, D80.1; no longer D10.C, D16.C, D22.C, D28.C, D34.C, D4.C, D40.C, D46.C, D52.C, D58.C, D64.C, D70.C, D75.C, D80.C
- net R5: now also D11.1, D17.1, D23.1, D29.1, D35.1, D41.1, D47.1, D5.1, D53.1, D59.1, D65.1, D71.1, D76.1, D81.1; no longer D11.C, D17.C, D23.C, D29.C, D35.C, D41.C, D47.C, D5.C, D53.C, D59.C, D65.C, D71.C, D76.C, D81.C
- net R6: now also D12.1, D18.1, D24.1, D30.1, D36.1, D42.1, D48.1, D54.1, D6.1, D60.1, D66.1; no longer D12.C, D18.C, D24.C, D30.C, D36.C, D42.C, D48.C, D54.C, D6.C, D60.C, D66.C
- net TDI: now also TP6.TP, U1.44
Routing:
- net TDI: track 0.00 -> 97.3 mm, vias 0 -> 4
- net R1: track 512.5 -> 491.4 mm, vias 0 -> 4
- net R3: track 470.3 -> 451.1 mm
- net R5: track 461.5 -> 476.1 mm, vias 4 -> 2
- net R4: track 458.9 -> 471.3 mm
- net N$120: track 0.00 -> 12.2 mm
- net N$119: track 0.00 -> 9.07 mm
- net N$113: track 0.00 -> 8.83 mm
- net N$27: track 39.6 -> 31.3 mm
- net N$114: track 0.00 -> 7.93 mm
- net R6: track 431.1 -> 438.9 mm
- net N$116: track 0.00 -> 7.41 mm
- net N$118: track 0.00 -> 7.19 mm
- net VREG_OUT: track 16.8 -> 23.9 mm, vias 0 -> 2
- net N$117: track 0.00 -> 7.06 mm
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Other:
- board text added: "80%"
