File: 80%/rev0.1x.brd (EAGLE design)
At the start: 375.5 x 123.8 mm, 208 parts, among them J1 USB-B, Q1 48MHz, SW1 CHERRY_MX, SW10 CHERRY_MX, SW11 CHERRY_MX, SW12 CHERRY_MX, SW13 CHERRY_MX, SW14 CHERRY_MX, SW15 CHERRY_MX, SW16 CHERRY_MX, SW17 CHERRY_MX, SW18 CHERRY_MX, SW19 CHERRY_MX, SW2 CHERRY_MX, SW20 CHERRY_MX, SW21 CHERRY_MX, SW22 CHERRY_MX, SW23 CHERRY_MX, SW24 CHERRY_MX, SW25 CHERRY_MX, SW26 CHERRY_MX, SW27 CHERRY_MX, SW28 CHERRY_MX, SW29 CHERRY_MX, SW3 CHERRY_MX, SW30 CHERRY_MX, SW31 CHERRY_MX, SW32 CHERRY_MX, SW33 CHERRY_MX, SW34 CHERRY_MX, SW35 CHERRY_MX, SW36 CHERRY_MX, SW37 CHERRY_MX, SW38 CHERRY_MX, SW39 CHERRY_MX, SW4 CHERRY_MX, SW40 CHERRY_MX, SW41 CHERRY_MX, SW42 CHERRY_MX, SW43 CHERRY_MX, SW44 CHERRY_MX, SW45 CHERRY_MX, SW46 CHERRY_MX, SW47 CHERRY_MX, SW48 CHERRY_MX, SW49 CHERRY_MX, SW5 CHERRY_MX, SW50 CHERRY_MX, SW51 CHERRY_MX, SW52 CHERRY_MX, SW53 CHERRY_MX, SW54 CHERRY_MX, SW55 CHERRY_MX, SW56 CHERRY_MX, SW57 CHERRY_MX, SW58 CHERRY_MX, SW59 CHERRY_MX, SW6 CHERRY_MX, SW60 CHERRY_MX, SW61 CHERRY_MX, SW62 CHERRY_MX, SW63 CHERRY_MX, SW64 CHERRY_MX, SW65 CHERRY_MX, SW66 CHERRY_MX, SW67 CHERRY_MX, SW68 CHERRY_MX, SW69 CHERRY_MX, SW7 CHERRY_MX, SW70 CHERRY_MX, SW71 CHERRY_MX, SW72 CHERRY_MX, SW73 CHERRY_MX, SW74 CHERRY_MX, SW75 CHERRY_MX, SW76 CHERRY_MX, SW77 CHERRY_MX, SW78 CHERRY_MX, SW79 CHERRY_MX, SW8 CHERRY_MX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

Commit message: closer to clean
Parts:
- moved C1 124.0 mm to (439.5, 181.6)
- moved C2 120.8 mm to (439.5, 183.8)
- moved C3 117.7 mm to (439.5, 185.9)
- moved C5 106.2 mm to (460.8, 197.1)
- moved C6 106.2 mm to (460.8, 203.5)
- moved C4 106.2 mm to (460.8, 190.8)
- moved C7 95.6 mm to (430.3, 173.7)
- moved C12 80.7 mm to (433.3, 183.6)
- moved C8 78.4 mm to (439.2, 163.3), turned to 270 degrees
- moved C9 74.9 mm to (452.4, 179.8), turned to 0 degrees
- moved C10 68.9 mm to (452.4, 177.5), turned to 0 degrees
- moved C11 66.4 mm to (448.8, 175.3), turned to 90 degrees
- moved TP1 60.0 mm to (448.8, 185.7)
- moved C13 55.8 mm to (448.8, 170.7), turned to 270 degrees
- moved SJ1 39.9 mm to (447.3, 182.4)
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Routing:
- net RESET: track 0.00 -> 65.5 mm
- net SWCLK: track 0.00 -> 61.0 mm
- net SWDIO: track 0.00 -> 48.9 mm
- net SWO: track 0.00 -> 32.2 mm
- net VCC3V3: track 0.00 -> 27.8 mm
- net N$2: track 0.00 -> 17.6 mm
- net VBUS1: track 0.00 -> 14.0 mm
- net USB1_P: track 15.3 -> 22.1 mm
- net USB1_N: track 15.1 -> 21.6 mm
